Commit message: "usd updated"

File: assets/urdf/dobot_magician_suction.urdf (robot description, URDF)
Before this commit: robot magician, 8 links, 7 joints
Links:
- link magician_base_link: mass None -> 1.0; geometry collision mesh filename=dobot_description/meshes/dae/magicianBase.dae; visual mesh filename=dobot_description/meshes/dae/magicianBase.dae
- link magician_link_1: mass None -> 0.5; geometry collision mesh filename=dobot_description/meshes/dae/magicianLink1.dae; visual mesh filename=dobot_description/meshes/dae/magicianLink1.dae
- link magician_link_2: mass None -> 0.3; geometry collision mesh filename=dobot_description/meshes/dae/magicianLink2.dae; visual mesh filename=dobot_description/meshes/dae/magicianLink2.dae
- link magician_link_3: mass None -> 0.3; geometry collision mesh filename=dobot_description/meshes/dae/magicianLink3.dae; visual mesh filename=dobot_description/meshes/dae/magicianLink3.dae
- link magician_link_4: mass None -> 0.1; geometry collision mesh filename=dobot_description/meshes/dae/magicianLink4.dae; visual mesh filename=dobot_description/meshes/dae/magicianLink4.dae
- link magician_link_suction_cup: mass None -> 0.05; geometry collision mesh filename=dobot_description/meshes/dae/suction_cup.dae; visual mesh filename=dobot_description/meshes/dae/suction_cup.dae
- link magician_link_virtual: mass None -> 0.01
